File: planck.kicad_sch (KiCad schematic)
At the start: 54 parts, among them J1 C128990, J2 USB_C_U262-161N-4BVC11, J3 C128990, SW1 SW_Cherry_MX_1.00u, SW10 SW_Cherry_MX_1.00u, SW11 SW_Cherry_MX_1.00u, SW12 SW_Cherry_MX_1.00u, SW13 SW_Cherry_MX_1.00u, SW14 SW_Cherry_MX_1.00u, SW15 SW_Cherry_MX_1.00u, SW16 SW_Cherry_MX_1.00u, SW17 SW_Cherry_MX_1.00u, SW18 SW_Cherry_MX_1.00u, SW19 SW_Cherry_MX_1.00u, SW2 SW_Cherry_MX_1.00u, SW20 SW_Cherry_MX_1.00u, SW21 SW_Cherry_MX_1.00u, SW22 SW_Cherry_MX_1.00u, SW23 SW_Cherry_MX_1.00u, SW24 SW_Cherry_MX_1.00u, SW3 SW_Cherry_MX_1.00u, SW4 SW_Cherry_MX_1.00u, SW5 SW_Cherry_MX_1.00u, SW6 SW_Cherry_MX_1.00u, SW7 SW_Cherry_MX_1.00u, SW8 SW_Cherry_MX_1.00u, SW9 SW_Cherry_MX_1.00u, U2 RP2040

Commit message: some modifications
Parts:
- removed J1, J3: C128990, C128990:C128990_3.5MM_TRRS, symbol C128990:C128990
- removed U2: RP2040, RP2040_minimal:RP2040-QFN-56, symbol MCU_RaspberryPi_and_Boards:RP2040
- added J1: USB_C_U262-161N-4BVC11, josh-connectors:USB_C_U262-161N-4BVC11, symbol josh-connector:USB_C_U262-161N-4BVC11
- added R3, R4, R5, R6: 100r 0201, Resistor_SMD:R_0201_0603Metric, symbol Device:R
- added U1: RP2040, RP2040_minimal:RP2040-QFN-56, symbol MCU_RaspberryPi_and_Boards:RP2040
- added Y1: 32M, Crystal:Crystal_SMD_3225-4Pin_3.2x2.5mm, symbol Device:Crystal_GND24
Connections:
- net GND: now also J1.A1 (GND), J1.A12 (GND), J1.B1 (GND), J1.B12 (GND), J1.S1 (SHIELD), Y1.2, Y1.4
- net VBUS: now also J1.A4 (VBUS), J1.A9 (VBUS), J1.B4 (VBUS), J1.B9 (VBUS)
- new net: J1.A6 (D+), J1.B6 (D+), R3.1, R5.1
- new net: J1.A7 (D-), J1.B7 (D-), R4.1, R6.1
- new net X32MI: Y1.1
- new net X32MO: Y1.3
- new net dx0: R5.2, R6.2
- new net tx0: R3.2, R4.2
- no-connect marks 2 -> 4
Other:
- moved on the sheet: J2, R1, R2

Commit message: MX version complete
Parts:
- added C1, C2: 2.2uF ±10% 10V, Resistor_SMD:R_0201_0603Metric, symbol Device:C
- added C10, C11, C12, C13, C15, C16, C5, C7, C8, C9: 100nF ±10% 25V 0201, Resistor_SMD:R_0201_0603Metric, symbol Device:C
- added C14, C6: 1uF ±20% 6.3V 0201, Capacitor_SMD:C_0201_0603Metric, symbol Device:C
- added C3, C4: 22pF ±5% 50V 0603, Resistor_SMD:R_0201_0603Metric, symbol Device:C
- added H1, H2, H3, H4: MountingHole, MountingHole:MountingHole_2.7mm_M2.5, symbol Mechanical:MountingHole
- added R7: 100Ω ±1% 50mW, Resistor_SMD:R_0201_0603Metric, symbol Device:R
- added R8: 10kΩ ±1% 50mW 0201, Resistor_SMD:R_0201_0603Metric, symbol Device:R
- added R9: 1kΩ ±1% 50mW 0201, Resistor_SMD:R_0201_0603Metric, symbol Device:R
- added SW25: SW_Push, symbol Switch:SW_Push
- added U2: ME6219C33M5G, Package_TO_SOT_SMD:SOT-23-5, symbol MCU_RaspberryPi_and_Boards:ME6219C33M5G
- added U3: W25Q16JVUXIQ, Package_SON:SON-8-1EP_3x2mm_P0.5mm_EP1.4x1.6mm, symbol W25Q16JVSSIQ:W25Q16JVSSIQ
- D1, D10, D11, D12, D13, D14, D15, D16, D17, D18, D19, D2, D20, D21, D22, D23, D24, D3, D4, D5, D6, D7, D8, D9: value 1N4148W -> 1N4148W,100V 150mA 4ns T4; JLC (none) -> C2099
- J1, J2: footprint josh-connectors:USB_C_U262-161N-4BVC11 -> josh-connectors:USB_C_TYPE-C-31-M-14; JLC (none) -> C319148; LCSC C319148 -> (none)
- R1, R2: JLC (none) -> C473460
- R3: value 100r 0201 -> 1kΩ ±1% 50mW 0201; JLC (none) -> C138165
- R4: value 100r 0201 -> 100Ω ±1% 50mW; JLC (none) -> C77623
- R5, R6: value 100r 0201 -> 27Ω ±1% 50mW 0201; JLC (none) -> C273268
- U1: value RP2040 -> RP2040 ARM Cortex-M0 133MHz; footprint RP2040_minimal:RP2040-QFN-56 -> Package_DFN_QFN:QFN-56-1EP_7x7mm_P0.4mm_EP3.2x3.2mm_ThermalVias; JLC (none) -> C2040
- Y1: value 32M -> 32MHz ±10ppm 20pF SMD3225-4P; JLC (none) -> C164054; jlc C164054 -> (none)
Connections:
- net GND: now also U1.19 (TESTEN), U1.57 (GND), C1.2, C10.1, C11.1, C12.1, C13.1, C14.1, C15.2, C16.2, C2.2, C3.2, C4.2, C5.1, C6.2, C7.1, C8.1, C9.1, SW25.1, U2.2 (GND), U3.4 (GND), U3.9 (EXP)
- net VBUS: now also C1.1, U2.1 (VIN), U2.3 (EN)
- net X32MI: now also U1.20 (XIN), C3.1
- net X32MO: now also R3.2, U1.21 (XOUT); no longer Y1.3
- net c1: now also U1.32 (GPIO21)
- net c2: now also U1.31 (GPIO20)
- net c3: now also U1.30 (GPIO19)
- net c4: now also U1.16 (GPIO13)
- net c5: now also U1.15 (GPIO12)
- net c6: now also U1.14 (GPIO11)
- net r1: now also U1.4 (GPIO2)
- net r2: now also U1.5 (GPIO3)
- net r3: now also U1.29 (GPIO18)
- net r4: now also U1.28 (GPIO17)
- net tx0: now also U1.2 (GPIO0); no longer R3.2
- net at J1.A6 (D+), J1.B6 (D+): now also R7.1; no longer R3.1, R5.1
- net V3V3: now reaches U1.1 (IOVDD)
- net V3V3: now also U1.10 (IOVDD), U1.22 (IOVDD), U1.33 (IOVDD), U1.42 (IOVDD), U1.43 (ADC_AVDD), U1.44 (VREG_IN), U1.48 (USB_VDD), U1.49 (IOVDD), C10.2, C11.2, C12.2, C13.2, C2.1, C6.1, C7.2, C8.2, C9.2, U2.5 (VOUT)
- net V1V1: now reaches U1.23 (DVDD)
- net V1V1: now also U1.45 (VREG_VOUT), U1.50 (DVDD), C14.2, C15.1, C16.1
- net rx0: now reaches U1.3 (GPIO1)
- net rx0: now also R7.2
- net at U1.46 (USB_DM): now also R6.1
- net at U1.47 (USB_DP): now also R5.1
- net QSPI_SD3: now reaches U1.51 (QSPI_SD3)
- net QSPI_SD3: now also U3.7 (IO3)
- net QSPI_CLK: now reaches U1.52 (QSPI_SCLK)
- net QSPI_CLK: now also U3.6 (CLK)
- net QSPI_SD0: now reaches U1.53 (QSPI_SD0)
- net QSPI_SD0: now also U3.5 (DI(IO0))
- net QSPI_SD2: now reaches U1.54 (QSPI_SD2)
- net QSPI_SD2: now also U3.3 (IO2)
- net QSPI_SD1: now reaches U1.55 (QSPI_SD1)
- net QSPI_SD1: now also U3.2 (DO(IO1))
- net QSPI_SS: now reaches U1.56 (QSPI_SS)
- net QSPI_SS: now also R8.1, R9.2, U3.1 (~{CS})
- net at J1.A7 (D-), J1.B7 (D-), R4.1: no longer R6.1
- net d+ renamed D-
- net D-: now also R5.2
- net d- renamed D+
- net D+: now also R6.2
- removed net dx0: R5.2, R6.2
- new net: C5.2, R8.2, U3.8 (VCC)
- new net: C4.1, R3.1, Y1.3
- new net: R9.1, SW25.2
- no-connect marks 4 -> 6
Other:
- moved on the sheet: R1, R2, U1, Y1

Commit message: add choc libraries
Parts:
- SW1, SW10, SW11, SW12, SW13, SW14, SW15, SW16, SW17, SW18, SW19, SW2, SW20, SW21, SW22, SW23, SW24, SW3, SW4, SW5, SW6, SW7, SW8, SW9: footprint Switches:SW_Cherry_MX_1.00u_Plate_HS -> Switch_Keyboard_Hotswap_Kailh:SW_Hotswap_Kailh_Choc_V1V2
- U1: footprint Package_DFN_QFN:QFN-56-1EP_7x7mm_P0.4mm_EP3.2x3.2mm_ThermalVias -> MCU_RaspberryPi_and_Boards:RP2040-QFN-56

Commit message: core board sketch
Parts:
- removed C1, C2: 2.2uF ±10% 10V, Resistor_SMD:R_0201_0603Metric, symbol Device:C
- removed D1, D10, D11, D12, D13, D14, D15, D16, D17, D18, D19, D2, D20, D21, D22, D23, D24, D3, D4, D5, D6, D7, D8, D9: 1N4148W,100V 150mA 4ns T4, Diode_SMD:D_SOD-123, symbol Diode:1N4148W
- removed H1, H2, H3, H4: MountingHole, MountingHole:MountingHole_2.7mm_M2.5, symbol Mechanical:MountingHole
- removed J1, J2: USB_C_U262-161N-4BVC11, josh-connectors:USB_C_TYPE-C-31-M-14, symbol josh-connector:USB_C_U262-161N-4BVC11
- removed R1, R2: 5.1k 0201, Resistor_SMD:R_0201_0603Metric, symbol Device:R
- removed R4, R7: 100Ω ±1% 50mW, Resistor_SMD:R_0201_0603Metric, symbol Device:R
- removed SW1, SW10, SW11, SW12, SW13, SW14, SW15, SW16, SW17, SW18, SW19, SW2, SW20, SW21, SW22, SW23, SW24, SW3, SW4, SW5, SW6, SW7, SW8, SW9: SW_Cherry_MX_1.00u, Switch_Keyboard_Hotswap_Kailh:SW_Hotswap_Kailh_Choc_V1V2, symbol Switches:SW_Cherry_MX_1.00u
- removed U2: ME6219C33M5G, Package_TO_SOT_SMD:SOT-23-5, symbol MCU_RaspberryPi_and_Boards:ME6219C33M5G
Connections:
- no-connect marks 6 -> 2
