File: planck.kicad_sch (KiCad schematic)
At the start: 129 parts, among them J2 USB_C_U262-161N-4BVC11, SW1 SW_Hotswap_Kailh_Choc_V1_1u, SW10 SW_Hotswap_Kailh_Choc_V1_1u, SW11 SW_Hotswap_Kailh_Choc_V1_1u, SW12 SW_Hotswap_Kailh_Choc_V1_1u, SW13 SW_Hotswap_Kailh_Choc_V1_1u, SW14 SW_Hotswap_Kailh_Choc_V1_1u, SW15 SW_Hotswap_Kailh_Choc_V1_1u, SW16 SW_Hotswap_Kailh_Choc_V1_1u, SW17 SW_Hotswap_Kailh_Choc_V1_1u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

Commit message: layout
Parts:
- added J1, J3: USB_C_U262-161N-4BVC11, josh-connectors:USB_C_TYPE-C-31-M-14, symbol josh-connector:USB_C_U262-161N-4BVC11
- D25, D26, D29, D30, D31, D32, D35, D36, D37, D38, D41, D42, D43, D44, D45, D46, D47, D48: footprint MCU_RaspberryPi_and_Boards:WS2812_6028_REV -> MCU_RaspberryPi_and_Boards:WS2812_6028_REV_S
Connections:
- net GND: now also J1.A1 (GND), J1.A12 (GND), J1.B1 (GND), J1.B12 (GND), J1.S1 (SHIELD), J3.A1 (GND), J3.A12 (GND), J3.B1 (GND), J3.B12 (GND), J3.S1 (SHIELD)
- net c3: now also U1.29 (GPIO18); no longer U1.30 (GPIO19)
- net c4: now also U1.9 (GPIO7); no longer U1.16 (GPIO13)
- net c6: now also U1.8 (GPIO6); no longer U1.14 (GPIO11)
- net r1: now also U1.37 (GPIO25); no longer U1.4 (GPIO2)
- net r2: now also U1.7 (GPIO5); no longer U1.5 (GPIO3)
- net r3: now also SW13.1, U1.34 (GPIO22); no longer SW13.2, U1.29 (GPIO18)
- net r4: now also SW19.2, SW20.2, SW21.2, SW22.2, SW23.2; no longer SW19.1, SW20.1, SW21.1, SW22.1, SW23.1
- net at D20.1 (K): now also SW20.1; no longer SW20.2
- net at D13.1 (K): now also SW13.2; no longer SW13.1
- net at D21.1 (K): now also SW21.1; no longer SW21.2
- net at D19.1 (K): now also SW19.1; no longer SW19.2
- net at D22.1 (K): now also SW22.1; no longer SW22.2
- net at D23.1 (K): now also SW23.1; no longer SW23.2
- new net: J3.A4 (VBUS), J3.A9 (VBUS), J3.B4 (VBUS), J3.B9 (VBUS)
- new net: J1.A4 (VBUS), J1.A9 (VBUS), J1.B4 (VBUS), J1.B9 (VBUS)
Other:
- moved on the sheet: C10, C11, C12, C13, C14, C15, C16, C3, C4, C6, C7, C8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

Commit message: layout
Connections:
- net VBUS: now also J1.A4 (VBUS), J1.A9 (VBUS), J1.B4 (VBUS), J1.B9 (VBUS), J3.A4 (VBUS), J3.A9 (VBUS), J3.B4 (VBUS), J3.B9 (VBUS)
- net rx0: now also J1.A6 (D+), J1.B6 (D+), J3.A7 (D-), J3.B7 (D-)
- net tx0: now also J1.A7 (D-), J1.B7 (D-), J3.A6 (D+), J3.B6 (D+)
Changed lines of the file:
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@@
   (junction (at 87.63 151.13) (diameter 0) (color 0 0 0 0)
   )
+  (junction (at 383.54 87.63) (diameter 0) (color 0 0 0 0)
+  )
   (junction (at 144.78 101.6) (diameter 0) (color 0 0 0 0)
   )
@@
   (junction (at 172.72 270.51) (diameter 0) (color 0 0 0 0)
   )
+  (junction (at 337.82 87.63) (diameter 0) (color 0 0 0 0)
+  )
   (junction (at 33.02 257.81) (diameter 0) (color 0 0 0 0)
   )
@@
   (junction (at 187.96 270.51) (diameter 0) (color 0 0 0 0)
   )
+  (junction (at 337.82 90.17) (diameter 0) (color 0 0 0 0)
+  )
   (junction (at 39.37 238.76) (diameter 0) (color 0 0 0 0)
   )
@@
   )
   (junction (at 86.36 215.9) (diameter 0) (color 0 0 0 0)
+  )
+  (junction (at 383.54 90.17) (diameter 0) (color 0 0 0 0)
   )
   (junction (at 269.24 36.83) (diameter 0) (color 0 0 0 0)
@@
     (stroke (width 0) (type default))
   )
+  (wire (pts (xy 377.19 87.63) (xy 383.54 87.63))
+    (stroke (width 0) (type default))
+  )
   (wire (pts (xy 118.11 101.6) (xy 118.11 125.73))
     (stroke (width 0) (type default))
@@
     (stroke (width 0) (type default))
   )
+  (wire (pts (xy 331.47 90.17) (xy 337.82 90.17))
+    (stroke (width 0) (type default))
+  )
   (wire (pts (xy 163.83 218.44) (xy 29.21 218.44))
     (stroke (width 0) (type default))
@@
     (stroke (width 0) (type default))
   )
+  (wire (pts (xy 337.82 85.09) (xy 331.47 85.09))
+    (stroke (width 0) (type default))
+  )
+  (wire (pts (xy 344.17 87.63) (xy 337.82 87.63))
+    (stroke (width 0) (type default))
+  )
   (wire (pts (xy 106.68 215.9) (xy 130.81 215.9))
     (stroke (width 0) (type default))
@@
     (stroke (width 0) (type default))
   )
+  (wire (pts (xy 383.54 87.63) (xy 383.54 85.09))
+    (stroke (width 0) (type default))
+  )
   (wire (pts (xy 242.57 151.13) (xy 233.68 151.13))
     (stroke (width 0) (type default))
@@
     (stroke (width 0) (type default))
   )
+  (wire (pts (xy 383.54 90.17) (xy 383.54 92.71))
+    (stroke (width 0) (type default))
+  )
   (wire (pts (xy 229.87 191.77) (xy 231.14 191.77))
     (stroke (width 0) (type default))
@@
     (stroke (width 0) (type default))
   )
+  (wire (pts (xy 377.19 72.39) (xy 383.54 72.39))
+    (stroke (width 0) (type default))
+  )
   (wire (pts (xy 166.37 67.31) (xy 167.64 67.31))
     (stroke (width 0) (type default))
@@
     (stroke (width 0) (type default))
   )
+  (wire (pts (xy 377.19 90.17) (xy 383.54 90.17))
+    (stroke (width 0) (type default))
+  )
   (wire (pts (xy 379.73 137.16) (xy 379.73 140.97))
     (stroke (width 0) (type default))
@@
     (stroke (width 0) (type default))
   )
+  (wire (pts (xy 337.82 87.63) (xy 337.82 85.09))
+    (stroke (width 0) (type default))
+  )
   (wire (pts (xy 172.72 270.51) (xy 172.72 267.97))
     (stroke (width 0) (type default))
@@
     (stroke (width 0) (type default))
   )
+  (wire (pts (xy 383.54 85.09) (xy 377.19 85.09))
+    (stroke (width 0) (type default))
+  )
   (wire (pts (xy 41.91 115.57) (xy 44.45 115.57))
     (stroke (width 0) (type default))
@@
     (stroke (width 0) (type default))
   )
+  (wire (pts (xy 383.54 92.71) (xy 377.19 92.71))
+    (stroke (width 0) (type default))
+  )
   (wire (pts (xy 237.49 215.9) (xy 243.84 215.9))
     (stroke (width 0) (type default))
@@
     (stroke (width 0) (type default))
   )
+  (wire (pts (xy 344.17 90.17) (xy 337.82 90.17))
+    (stroke (width 0) (type default))
+  )
   (wire (pts (xy 128.27 73.66) (xy 125.73 73.66))
     (stroke (width 0) (type default))
@@
     (stroke (width 0) (type default))
   )
+  (wire (pts (xy 331.47 87.63) (xy 337.82 87.63))
+    (stroke (width 0) (type default))
+  )
   (wire (pts (xy 140.97 270.51) (xy 148.59 270.51))
     (stroke (width 0) (type default))
@@
     (stroke (width 0) (type default))
   )
+  (wire (pts (xy 331.47 72.39) (xy 337.82 72.39))
+    (stroke (width 0) (type default))
+  )
   (wire (pts (xy 121.92 43.18) (xy 124.46 43.18))
     (stroke (width 0) (type default))
@@
     (stroke (width 0) (type default))
   )
+  (wire (pts (xy 389.89 87.63) (xy 383.54 87.63))
+    (stroke (width 0) (type default))
+  )
   (wire (pts (xy 132.08 173.99) (xy 154.94 173.99))
     (stroke (width 0) (type default))
@@
     (stroke (width 0) (type default))
   )
+  (wire (pts (xy 389.89 90.17) (xy 383.54 90.17))
+    (stroke (width 0) (type default))
+  )
   (wire (pts (xy 288.29 144.78) (xy 288.29 137.16))
     (stroke (width 0) (type default))
@@
     (stroke (width 0) (type default))
   )
+  (wire (pts (xy 337.82 92.71) (xy 331.47 92.71))
+    (stroke (width 0) (type default))
+  )
   (wire (pts (xy 189.23 97.79) (xy 194.31 97.79))
     (stroke (width 0) (type default))
@@
     (stroke (width 0) (type default))
   )
+  (wire (pts (xy 337.82 90.17) (xy 337.82 92.71))
+    (stroke (width 0) (type default))
+  )
   (wire (pts (xy 373.38 52.07) (xy 375.92 52.07))
     (stroke (width 0) (type default))
@@
     (effects (font (size 1.27 1.27)) (justify left bottom))
   )
+  (label "VBUS" (at 332.74 72.39 0) (fields_autoplaced)
+    (effects (font (size 1.27 1.27)) (justify left bottom))
+  )
   (label "V3V3" (at 370.84 24.13 0) (fields_autoplaced)
     (effects (font (size 1.27 1.27)) (justify left bottom))
   )
+  (label "rx0" (at 384.81 87.63 0) (fields_autoplaced)
+    (effects (font (size 1.27 1.27)) (justify left bottom))
+  )
   (label "QSPI_SD3" (at 331.47 52.07 0) (fields_autoplaced)
     (effects (font (size 1.27 1.27)) (justify left bottom))
@@
     (effects (font (size 1.27 1.27)) (justify left bottom))
   )
+  (label "rx0" (at 340.36 90.17 0) (fields_autoplaced)
+    (effects (font (size 1.27 1.27)) (justify left bottom))
+  )
   (label "VBUS" (at 77.47 173.99 0) (fields_autoplaced)
     (effects (font (size 1.27 1.27)) (justify left bottom))
   )
+  (label "tx0" (at 384.81 90.17 0) (fields_autoplaced)
+    (effects (font (size 1.27 1.27)) (justify left bottom))
+  )
   (label "QSPI_SD0" (at 248.9189 167.64 0) (fields_autoplaced)
     (effects (font (size 1.27 1.27)) (justify left bottom))
@@
     (effects (font (size 1.27 1.27)) (justify left bottom))
   )
+  (label "VBUS" (at 378.46 72.39 0) (fields_autoplaced)
+    (effects (font (size 1.27 1.27)) (justify left bottom))
+  )
   (label "D+" (at 254 49.53 0) (fields_autoplaced)
     (effects (font (size 1.27 1.27)) (justify left bottom))
@@
     (effects (font (size 1.27 1.27)) (justify left bottom))
   )
+  (label "tx0" (at 340.36 87.63 0) (fields_autoplaced)
+    (effects (font (size 1.27 1.27)) (justify left bottom))
+  )
