File: planck.kicad_pcb (KiCad board)
At the start: 2 copper layers, 115 x 75 mm, 131 parts, among them J1 USB_C_U262-161N-4BVC11, J2 USB_C_U262-161N-4BVC11, J3 USB_C_U262-161N-4BVC11, SW1 SW_Hotswap_Kailh_Choc_V1_1u, SW10 SW_Hotswap_Kailh_Choc_V1_1u, SW11 SW_Hotswap_Kailh_Choc_V1_1u, SW12 SW_Hotswap_Kailh_Choc_V1_1u, SW13 SW_Hotswap_Kailh_Choc_V1_1u, SW14 SW_Hotswap_Kailh_Choc_V1_1u, SW15 SW_Hotswap_Kailh_Choc_V1_1u, SW16 SW_Hotswap_Kailh_Choc_V1_1u, SW17 SW_Hotswap_Kailh_Choc_V1_1u, SW18 SW_Hotswap_Kailh_Choc_V1_1u, SW19 SW_Hotswap_Kailh_Choc_V1_1u, SW2 SW_Hotswap_Kailh_Choc_V1_1u, SW20 SW_Hotswap_Kailh_Choc_V1_1u, SW21 SW_Hotswap_Kailh_Choc_V1_1u, SW22 SW_Hotswap_Kailh_Choc_V1_1u, SW23 SW_Hotswap_Kailh_Choc_V1_1u, SW24 SW_Hotswap_Kailh_Choc_V1_1u, SW25 SW_Push, SW3 SW_Hotswap_Kailh_Choc_V1_1u, SW4 SW_Hotswap_Kailh_Choc_V1_1u, SW5 SW_Hotswap_Kailh_Choc_V1_1u, SW6 SW_Hotswap_Kailh_Choc_V1_1u, SW7 SW_Hotswap_Kailh_Choc_V1_1u, SW8 SW_Hotswap_Kailh_Choc_V1_1u, SW9 SW_Hotswap_Kailh_Choc_V1_1u, U1 RP2040 ARM Cortex-M0 133MHz, U2 ME6219C33M5G, U3 W25Q16JVUXIQ, Y1 32MHz ±10ppm 20pF SMD3225-4P

Commit message: layout
Parts:
- D25, D26, D29, D30, D31, D32, D35, D36, D37, D38, D41, D42, D43, D44, D45, D46, D47, D48: footprint MCU_RaspberryPi_and_Boards:WS2812_6028_REV -> MCU_RaspberryPi_and_Boards:WS2812_6028_REV_S
- moved C35 2.82 mm to (169.9, 61.7), turned to -90 degrees
- moved C21 2.74 mm to (94.0, 61.7), turned to -90 degrees
- moved C19 0.75 mm to (190.4, 101.4)
- moved C25 0.70 mm to (114.5, 101.6)
- moved C31 0.70 mm to (106.5, 131.4)
- moved C38 0.70 mm to (87.5, 131.4)
- moved C22 0.70 mm to (163.5, 93.5)
- moved C26 0.68 mm to (171.5, 101.6)
- moved C17 0.65 mm to (144.5, 131.4)
- moved C24 0.65 mm to (125.5, 131.6)
- moved C39 0.65 mm to (182.5, 131.4)
- moved C40 0.65 mm to (163.5, 131.4)
- moved C27 0.60 mm to (182.4, 93.6)
- moved C30 0.56 mm to (106.4, 93.5)
- moved C23 0.55 mm to (87.4, 93.6)
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Connections:
- J1 pad A4: Net-(J1-VBUS-PadA4) -> /VBUS
- J1 pad A6: unconnected-(J1-D+-PadA6) -> /rx0
- J1 pad A7: unconnected-(J1-D--PadA7) -> /tx0
- J1 pad A9: Net-(J1-VBUS-PadA4) -> /VBUS
- J1 pad B4: Net-(J1-VBUS-PadA4) -> /VBUS
- J1 pad B6: unconnected-(J1-D+-PadB6) -> /rx0
- J1 pad B7: unconnected-(J1-D--PadB7) -> /tx0
- J1 pad B9: Net-(J1-VBUS-PadA4) -> /VBUS
- J3 pad A4: Net-(J3-VBUS-PadA4) -> /VBUS
- J3 pad A6: unconnected-(J3-D+-PadA6) -> /tx0
- J3 pad A7: unconnected-(J3-D--PadA7) -> /rx0
- J3 pad A9: Net-(J3-VBUS-PadA4) -> /VBUS
- J3 pad B4: Net-(J3-VBUS-PadA4) -> /VBUS
- J3 pad B6: unconnected-(J3-D+-PadB6) -> /tx0
- J3 pad B7: unconnected-(J3-D--PadB7) -> /rx0
- J3 pad B9: Net-(J3-VBUS-PadA4) -> /VBUS
Routing:
- net /rx0: track 13.8 -> 264.6 mm, vias 0 -> 5
- net /tx0: track 14.0 -> 261.3 mm, vias 0 -> 5
- net /VBUS: track 584.4 -> 689.7 mm, vias 17 -> 26
- net Net-(D29-DOUT): track 15.1 -> 27.1 mm, vias 0 -> 4
- net Net-(D25-DOUT): track 14.9 -> 26.1 mm, vias 0 -> 4
- net Net-(D24-K): track 6.63 -> 9.04 mm
- net Net-(D31-DOUT): track 13.8 -> 15.2 mm
- net Net-(D41-DOUT): track 15.0 -> 15.9 mm
- net Net-(D43-DOUT): track 14.5 -> 15.3 mm
- net r1: track 154.8 -> 154.0 mm
- net Net-(D30-DOUT): track 40.5 -> 41.1 mm
- net GND: vias 7 -> 4
Other:
- outline, holes or cut-outs redrawn

Commit message: almost done
Parts:
- H1, H2, H3, H4: footprint MountingHole:MountingHole_2.7mm_M2.5 -> MountingHole:MountingHole_2.2mm_M2
- SW25: footprint Switches:TSC005A1618A03 -> Switches:B3U-1000P
- moved SW25 1.00 mm to (148.5, 97.5), turned to 90 degrees
Routing:
- net GND: track 6.27 -> 12.6 mm, vias 4 -> 113
- net Net-(R9-Pad1): track 8.73 -> 4.94 mm
- net /VBUS: track 689.7 -> 688.5 mm
Other:
- board text added: "SERIAL"
- board text added: "USB"

Commit message: ADD SWITCH HANDSET
Parts:
- added R4: 1kΩ ±1% 50mW 0201, Resistor_SMD:R_0201_0603Metric, B.Cu at (154.2, 94.9)
- added R7: 1kΩ ±1% 50mW 0201, Resistor_SMD:R_0201_0603Metric, B.Cu at (154.2, 94.2)
- added SW26: ~, Switches:DSHP02TSGET, B.Cu at (157.6, 97.5)
Connections:
- U1 pad 11: unconnected-(U1-GPIO8-Pad11) -> c5
- U1 pad 12: unconnected-(U1-GPIO9-Pad12) -> Net-(U1-GPIO9)
- U1 pad 13: unconnected-(U1-GPIO10-Pad13) -> Net-(U1-GPIO10)
- U1 pad 15: c5 -> unconnected-(U1-GPIO12-Pad15)
Routing:
- net /V3V3: track 29.2 -> 62.0 mm
- net Net-(U1-GPIO9): track 0.00 -> 17.1 mm
- net Net-(U1-GPIO10): track 0.00 -> 15.2 mm
- net Net-(R4-Pad1): track 0.00 -> 4.44 mm
- net Net-(R7-Pad1): track 0.00 -> 2.66 mm
- net GND: vias 113 -> 115
Other:
- board text added: "L/R"
